Commit message: robot falling in gazebo, tf not broadcasting

File: ws/install/gazebo_tools/share/gazebo_tools/description/my_robot.xacro (robot description, xacro)
@@ -1,7 +1,31 @@
 <?xml version="1.0"?>
-<robot name="example_robot" xmlns:xacro="http://www.ros.org/wiki/xacro">
-  <!-- Define macro before usage -->
+<robot name="my_robot" xmlns:xacro="http://www.ros.org/wiki/xacro">
+  <!-- Define the base link with inertia properties -->
+  <link name="base_link">
+    <visual>
+      <geometry>
+        <box size="0.5 0.5 0.1"/> <!-- Adjust size as needed -->
+      </geometry>
+      <material name="blue"/>
+    </visual>
+    <inertial>
+      <mass value="1.0"/> <!-- Mass in kg, make sure it's non-zero -->
+      <inertia ixx="0.01" ixy="0.0" ixz="0.0" iyy="0.01" iyz="0.0" izz="0.01"/> <!-- Inertia tensor -->
+    </inertial>
+  </link>
+  <!-- Define the first wheel with inertia properties -->
   <xacro:macro name="wheel" params="name">
-    <link name="${name}"/>
+    <link name="${name}">
+      <visual>
+        <geometry>
+          <cylinder length="0.05" radius="0.1"/> <!-- Adjust dimensions as needed -->
+        </geometry>
+        <material name="black"/>
+      </visual>
+      <inertial>
+        <mass value="0.1"/> <!-- Mass of the wheel -->
+        <inertia ixx="0.001" ixy="0.0" ixz="0.0" iyy="0.001" iyz="0.0" izz="0.001"/> <!-- Inertia tensor for the wheel -->
+      </inertial>
+    </link>
     <joint name="${name}_joint" type="continuous">
       <parent link="base_link"/>
