Commit message: teleop working

File: ws/install/gazebo_tools/share/gazebo_tools/description/my_robot.urdf.xacro (robot description, xacro)
@@ -1 +1,84 @@
-/ieee_simulation/ws/build/gazebo_tools/description/my_robot.urdf.xacro
+<?xml version="1.0"?>
+<robot name="my_robot" xmlns:xacro="http://www.ros.org/wiki/xacro">
+  <!-- Fixed map frame -->
+  <link name="map"/>
+  <!-- Base link with inertia properties -->
+  <link name="base_link">
+    <visual>
+      <geometry>
+        <box size="0.5 0.5 0.1"/> <!-- Adjust size as needed -->
+      </geometry>
+      <material name="blue"/>
+    </visual>
+    <inertial>
+      <mass value="1.0"/> <!-- Mass in kg, make sure it's non-zero -->
+      <inertia ixx="0.01" ixy="0.0" ixz="0.0" iyy="0.01" iyz="0.0" izz="0.01"/> <!-- Inertia tensor -->
+    </inertial>
+  </link>
+  <!-- Fixed joint between map and base_link -->
+  <joint name="map_to_base_link" type="fixed">
+    <parent link="map"/>
+    <child link="base_link"/>
+    <origin xyz="0 0 0" rpy="0 0 0"/> <!-- Adjust origin if needed -->
+  </joint>
+  <!-- Define the rotating wheel macro -->
+  <xacro:macro name="wheel" params="name position_x position_y">
+    <link name="${name}">
+      <visual>
+        <geometry>
+          <cylinder length="0.05" radius="0.1"/> <!-- Adjust dimensions as needed -->
+        </geometry>
+        <material name="black"/>
+      </visual>
+      <collision>
+        <geometry>
+          <cylinder length="0.05" radius="0.1"/>
+        </geometry>
+      </collision>
+      <inertial>
+        <mass value="0.1"/> <!-- Mass of the wheel -->
+        <inertia ixx="0.001" ixy="0.0" ixz="0.0" iyy="0.001" iyz="0.0" izz="0.001"/> <!-- Inertia tensor for the wheel -->
+      </inertial>
+    </link>
+    <!-- Continuous joint to allow rotation -->
+    <joint name="${name}_joint" type="continuous">
+      <parent link="base_link"/>
+      <child link="${name}"/>
+      <origin xyz="${position_x} ${position_y} 0.0" rpy="0 1.57 0"/> <!-- Position relative to base_link -->
+      <axis xyz="1 0 0"/> <!-- Wheel rotation around the Y-axis -->
+    </joint>
+    <!-- Transmission
+    <transmission name="${name}_transmission">
+      <type>simple_transmission</type>
+      <joint name="${name}_joint">
+        <hardwareInterface>hardware_interface/VelocityJointInterface</hardwareInterface>
+      </joint>
+      <actuator name="${name}_actuator">
+        <mechanicalReduction>1</mechanicalReduction>
+      </actuator>
+    </transmission> -->
+    <!-- ros2_control
+    <ros2_control>
+      <hardware>
+        <plugin>ignition_ros2_control/IgnitionSystem</plugin>
+      </hardware>
+      <joint name="${name}_joint">
+        <command_interfaces>velocity</command_interfaces>
+        <state_interfaces>position</state_interfaces>
+        <state_interfaces>velocity</state_interfaces>
+      </joint>
+    </ros2_control> -->
+  </xacro:macro>
+  <!-- Use the macro to create wheels -->
+  <!-- Front Left Wheel -->
+  <xacro:property name="wheel_offset_x" value="0.25"/> <!-- Front and rear offset along X -->
+  <xacro:property name="wheel_offset_y" value="0.20"/> <!-- Left and right offset along Y -->
+  <!-- Front Left Wheel -->
+  <xacro:wheel name="front_left_wheel" position_x="${wheel_offset_x}" position_y="${wheel_offset_y}"/>
+  <!-- Front Right Wheel -->
+  <xacro:wheel name="front_right_wheel" position_x="${wheel_offset_x}" position_y="-${wheel_offset_y}"/>
+  <!-- Rear Left Wheel -->
+  <xacro:wheel name="rear_left_wheel" position_x="-${wheel_offset_x}" position_y="${wheel_offset_y}"/>
+  <!-- Rear Right Wheel -->
+  <xacro:wheel name="rear_right_wheel" position_x="-${wheel_offset_x}" position_y="-${wheel_offset_y}"/>
+</robot>
