Commit message: updates to simulation in gazebo

File: ws/install/gazebo_tools/share/gazebo_tools/description/my_robot.urdf.xacro (robot description, xacro)
@@ -1,84 +1 @@
-<?xml version="1.0"?>
-<robot name="my_robot" xmlns:xacro="http://www.ros.org/wiki/xacro">
-  <!-- Fixed map frame -->
-  <link name="map"/>
-  <!-- Base link with inertia properties -->
-  <link name="base_link">
-    <visual>
-      <geometry>
-        <box size="0.5 0.5 0.1"/> <!-- Adjust size as needed -->
-      </geometry>
-      <material name="blue"/>
-    </visual>
-    <inertial>
-      <mass value="1.0"/> <!-- Mass in kg, make sure it's non-zero -->
-      <inertia ixx="0.01" ixy="0.0" ixz="0.0" iyy="0.01" iyz="0.0" izz="0.01"/> <!-- Inertia tensor -->
-    </inertial>
-  </link>
-  <!-- Fixed joint between map and base_link -->
-  <joint name="map_to_base_link" type="fixed">
-    <parent link="map"/>
-    <child link="base_link"/>
-    <origin xyz="0 0 0" rpy="0 0 0"/> <!-- Adjust origin if needed -->
-  </joint>
-  <!-- Define the rotating wheel macro -->
-  <xacro:macro name="wheel" params="name position_x position_y">
-    <link name="${name}">
-      <visual>
-        <geometry>
-          <cylinder length="0.05" radius="0.1"/> <!-- Adjust dimensions as needed -->
-        </geometry>
-        <material name="black"/>
-      </visual>
-      <collision>
-        <geometry>
-          <cylinder length="0.05" radius="0.1"/>
-        </geometry>
-      </collision>
-      <inertial>
-        <mass value="0.1"/> <!-- Mass of the wheel -->
-        <inertia ixx="0.001" ixy="0.0" ixz="0.0" iyy="0.001" iyz="0.0" izz="0.001"/> <!-- Inertia tensor for the wheel -->
-      </inertial>
-    </link>
-    <!-- Continuous joint to allow rotation -->
-    <joint name="${name}_joint" type="continuous">
-      <parent link="base_link"/>
-      <child link="${name}"/>
-      <origin xyz="${position_x} ${position_y} 0.0" rpy="0 1.57 0"/> <!-- Position relative to base_link -->
-      <axis xyz="1 0 0"/> <!-- Wheel rotation around the Y-axis -->
-    </joint>
-    <!-- Transmission
-    <transmission name="${name}_transmission">
-      <type>simple_transmission</type>
-      <joint name="${name}_joint">
-        <hardwareInterface>hardware_interface/VelocityJointInterface</hardwareInterface>
-      </joint>
-      <actuator name="${name}_actuator">
-        <mechanicalReduction>1</mechanicalReduction>
-      </actuator>
-    </transmission> -->
-    <!-- ros2_control
-    <ros2_control>
-      <hardware>
-        <plugin>ignition_ros2_control/IgnitionSystem</plugin>
-      </hardware>
-      <joint name="${name}_joint">
-        <command_interfaces>velocity</command_interfaces>
-        <state_interfaces>position</state_interfaces>
-        <state_interfaces>velocity</state_interfaces>
-      </joint>
-    </ros2_control> -->
-  </xacro:macro>
-  <!-- Use the macro to create wheels -->
-  <!-- Front Left Wheel -->
-  <xacro:property name="wheel_offset_x" value="0.25"/> <!-- Front and rear offset along X -->
-  <xacro:property name="wheel_offset_y" value="0.20"/> <!-- Left and right offset along Y -->
-  <!-- Front Left Wheel -->
-  <xacro:wheel name="front_left_wheel" position_x="${wheel_offset_x}" position_y="${wheel_offset_y}"/>
-  <!-- Front Right Wheel -->
-  <xacro:wheel name="front_right_wheel" position_x="${wheel_offset_x}" position_y="-${wheel_offset_y}"/>
-  <!-- Rear Left Wheel -->
-  <xacro:wheel name="rear_left_wheel" position_x="-${wheel_offset_x}" position_y="${wheel_offset_y}"/>
-  <!-- Rear Right Wheel -->
-  <xacro:wheel name="rear_right_wheel" position_x="-${wheel_offset_x}" position_y="-${wheel_offset_y}"/>
-</robot>
+/ieee_simulation/ws/build/gazebo_tools/description/my_robot.urdf.xacro

File: ws/src/gazebo_tools/description/BaseMecanumURDF_old.urdf.xacro (robot description, xacro)
@@ -8,14 +8,5 @@
       <visual>
         <origin xyz="0.0 0.0 0.0" rpy="0 0 0" />
-        <geometry>
-          <box size="0.1 0.1 0.1" />
-        </geometry>
       </visual>
-    <collision>
-      <origin xyz="0.0 0.0 0.0" rpy="0 0 0" />
-      <geometry>
-        <box size="0.1 0.1 0.1" />
-      </geometry>
-    </collision>
   </link>
   <!-- Joint to connect odom and base_link -->
@@ -47,5 +38,5 @@
       <geometry>
         <mesh
-          filename="package://gazebo_tools/meshes/robot/base_link.STL" />
+          filename="file://$(find gazebo_tools)/meshes/robot/base_link.STL" />
       </geometry>
       <material
@@ -61,5 +52,5 @@
       <geometry>
         <mesh
-          filename="package://gazebo_tools/meshes/robot/base_link.STL" />
+          filename="file://$(find gazebo_tools)/meshes/robot/base_link.STL" />
       </geometry>
     </collision>
@@ -81,11 +72,22 @@
         izz="9.1793540218031E-06" />
     </inertial>
-    <visual>
-      <origin
-        xyz="0 0 0"
-        rpy="0 0 0" />
-      <geometry>
-        <mesh
-          filename="package://gazebo_tools/meshes/robot/FrontRight_wheel.STL" />
+    <!-- <inertial>
+      <origin xyz="0 0 0" rpy="0 0 0" />
+      <mass value="0.0641393198112098" />
+      <inertia
+        ixx="0.0001"
+        ixy="0"
+        ixz="0"
+        iyy="0.0001"
+        iyz="0"
+        izz="0.0001" />
+    </inertial> -->
+    <!-- <visual>
+      <origin
+        xyz="0 0 0"
+        rpy="0 0 0" />
+      <geometry>
+        <mesh
+          filename="file://$(find gazebo_tools)/meshes/robot/FrontRight_wheel.STL" />
       </geometry>
       <material
@@ -94,12 +96,30 @@
           rgba="0.752941176470588 0.752941176470588 0.752941176470588 1" />
       </material>
-    </visual>
-    <collision>
-      <origin
-        xyz="0 0 0"
-        rpy="0 0 0" />
-      <geometry>
-        <mesh
-          filename="package://gazebo_tools/meshes/robot/FrontRight_wheel.STL" />
+    </visual>  -->
+    <!-- <collision>
+      <origin
+        xyz="-0.0200915998046353 -4.09353535379131E-05 -7.3187470010113E-05"
+        rpy="0 0 0" />
+       <geometry>
+        <mesh
+          filename="file://$(find gazebo_tools)/meshes/robot/FrontRight_wheel.STL" />
+      </geometry>
+      <geometry>
+        <cylinder radius="0.05" length="0.1"/>
+      </geometry>
+       <box size="0.5 0.3 0.1"/>
+    </collision> -->
+    <visual>
+      <origin
+        xyz="-0.02 0 0"
+        rpy="0 1.5708 0" />
+      <geometry>
+        <cylinder radius="0.04" length="0.03"/>
+      </geometry>
+    </visual>
+    <collision>
+      <origin xyz="0 0 0" rpy="0 0 0" />
+      <geometry>
+        <box size="0.04 0.04 0.04"/>
       </geometry>
     </collision>
@@ -140,19 +160,19 @@
       <geometry>
         <mesh
-          filename="package://gazebo_tools/meshes/robot/A_r1.STL" />
-      </geometry>
-      <material
-        name="">
-        <color
-          rgba="0.792156862745098 0.819607843137255 0.933333333333333 1" />
-      </material>
-    </visual>
-    <collision>
-      <origin
-        xyz="0 0 0"
-        rpy="0 0 0" />
-      <geometry>
-        <mesh
-          filename="package://gazebo_tools/meshes/robot/A_r1.STL" />
+          filename="file://$(find gazebo_tools)/meshes/robot/A_r1.STL" />
+      </geometry>
+      <material
+        name="">
+        <color
+          rgba="0.792156862745098 0.819607843137255 0.933333333333333 1" />
+      </material>
+    </visual>
+    <collision>
+      <origin
+        xyz="0 0 0"
+        rpy="0 0 0" />
+      <geometry>
+        <mesh
+          filename="file://$(find gazebo_tools)/meshes/robot/A_r1.STL" />
       </geometry>
     </collision>
@@ -193,19 +213,19 @@
       <geometry>
         <mesh
-          filename="package://gazebo_tools/meshes/robot/A_r2.STL" />
-      </geometry>
-      <material
-        name="">
-        <color
-          rgba="0.792156862745098 0.819607843137255 0.933333333333333 1" />
-      </material>
-    </visual>
-    <collision>
-      <origin
-        xyz="0 0 0"
-        rpy="0 0 0" />
-      <geometry>
-        <mesh
-          filename="package://gazebo_tools/meshes/robot/A_r2.STL" />
+          filename="file://$(find gazebo_tools)/meshes/robot/A_r2.STL" />
+      </geometry>
+      <material
+        name="">
+        <color
+          rgba="0.792156862745098 0.819607843137255 0.933333333333333 1" />
+      </material>
+    </visual>
+    <collision>
+      <origin
+        xyz="0 0 0"
+        rpy="0 0 0" />
+      <geometry>
+        <mesh
+          filename="file://$(find gazebo_tools)/meshes/robot/A_r2.STL" />
       </geometry>
     </collision>
@@ -246,19 +266,19 @@
       <geometry>
         <mesh
-          filename="package://gazebo_tools/meshes/robot/A_r3.STL" />
-      </geometry>
-      <material
-        name="">
-        <color
-          rgba="0.792156862745098 0.819607843137255 0.933333333333333 1" />
-      </material>
-    </visual>
-    <collision>
-      <origin
-        xyz="0 0 0"
-        rpy="0 0 0" />
-      <geometry>
-        <mesh
-          filename="package://gazebo_tools/meshes/robot/A_r3.STL" />
+          filename="file://$(find gazebo_tools)/meshes/robot/A_r3.STL" />
+      </geometry>
+      <material
+        name="">
+        <color
+          rgba="0.792156862745098 0.819607843137255 0.933333333333333 1" />
+      </material>
+    </visual>
+    <collision>
+      <origin
+        xyz="0 0 0"
+        rpy="0 0 0" />
+      <geometry>
+        <mesh
+          filename="file://$(find gazebo_tools)/meshes/robot/A_r3.STL" />
       </geometry>
     </collision>
@@ -299,19 +319,19 @@
       <geometry>
         <mesh
-          filename="package://gazebo_tools/meshes/robot/A_r4.STL" />
-      </geometry>
-      <material
-        name="">
-        <color
-          rgba="0.792156862745098 0.819607843137255 0.933333333333333 1" />
-      </material>
-    </visual>
-    <collision>
-      <origin
-        xyz="0 0 0"
-        rpy="0 0 0" />
-      <geometry>
-        <mesh
-          filename="package://gazebo_tools/meshes/robot/A_r4.STL" />
+          filename="file://$(find gazebo_tools)/meshes/robot/A_r4.STL" />
+      </geometry>
+      <material
+        name="">
+        <color
+          rgba="0.792156862745098 0.819607843137255 0.933333333333333 1" />
+      </material>
+    </visual>
+    <collision>
+      <origin
+        xyz="0 0 0"
+        rpy="0 0 0" />
+      <geometry>
+        <mesh
+          filename="file://$(find gazebo_tools)/meshes/robot/A_r4.STL" />
       </geometry>
     </collision>
@@ -352,19 +372,19 @@
       <geometry>
         <mesh
-          filename="package://gazebo_tools/meshes/robot/A_r5.STL" />
-      </geometry>
-      <material
-        name="">
-        <color
-          rgba="0.792156862745098 0.819607843137255 0.933333333333333 1" />
-      </material>
-    </visual>
-    <collision>
-      <origin
-        xyz="0 0 0"
-        rpy="0 0 0" />
-      <geometry>
-        <mesh
-          filename="package://gazebo_tools/meshes/robot/A_r5.STL" />
+          filename="file://$(find gazebo_tools)/meshes/robot/A_r5.STL" />
+      </geometry>
+      <material
+        name="">
+        <color
+          rgba="0.792156862745098 0.819607843137255 0.933333333333333 1" />
+      </material>
+    </visual>
+    <collision>
+      <origin
+        xyz="0 0 0"
+        rpy="0 0 0" />
+      <geometry>
+        <mesh
+          filename="file://$(find gazebo_tools)/meshes/robot/A_r5.STL" />
       </geometry>
     </collision>
@@ -405,19 +425,19 @@
       <geometry>
         <mesh
-          filename="package://gazebo_tools/meshes/robot/A_r6.STL" />
-      </geometry>
-      <material
-        name="">
-        <color
-          rgba="0.792156862745098 0.819607843137255 0.933333333333333 1" />
-      </material>
-    </visual>
-    <collision>
-      <origin
-        xyz="0 0 0"
-        rpy="0 0 0" />
-      <geometry>
-        <mesh
-          filename="package://gazebo_tools/meshes/robot/A_r6.STL" />
+          filename="file://$(find gazebo_tools)/meshes/robot/A_r6.STL" />
+      </geometry>
+      <material
+        name="">
+        <color
+          rgba="0.792156862745098 0.819607843137255 0.933333333333333 1" />
+      </material>
+    </visual>
+    <collision>
+      <origin
+        xyz="0 0 0"
+        rpy="0 0 0" />
+      <geometry>
+        <mesh
+          filename="file://$(find gazebo_tools)/meshes/robot/A_r6.STL" />
       </geometry>
     </collision>
@@ -458,19 +478,19 @@
       <geometry>
         <mesh
-          filename="package://gazebo_tools/meshes/robot/A_r7.STL" />
-      </geometry>
-      <material
-        name="">
-        <color
-          rgba="0.792156862745098 0.819607843137255 0.933333333333333 1" />
-      </material>
-    </visual>
-    <collision>
-      <origin
-        xyz="0 0 0"
-        rpy="0 0 0" />
-      <geometry>
-        <mesh
-          filename="package://gazebo_tools/meshes/robot/A_r7.STL" />
+          filename="file://$(find gazebo_tools)/meshes/robot/A_r7.STL" />
+      </geometry>
+      <material
+        name="">
+        <color
+          rgba="0.792156862745098 0.819607843137255 0.933333333333333 1" />
+      </material>
+    </visual>
+    <collision>
+      <origin
+        xyz="0 0 0"
+        rpy="0 0 0" />
+      <geometry>
+        <mesh
+          filename="file://$(find gazebo_tools)/meshes/robot/A_r7.STL" />
       </geometry>
     </collision>
@@ -511,19 +531,19 @@
       <geometry>
         <mesh
-          filename="package://gazebo_tools/meshes/robot/A_r8.STL" />
-      </geometry>
-      <material
-        name="">
-        <color
-          rgba="0.792156862745098 0.819607843137255 0.933333333333333 1" />
-      </material>
-    </visual>
-    <collision>
-      <origin
-        xyz="0 0 0"
-        rpy="0 0 0" />
-      <geometry>
-        <mesh
-          filename="package://gazebo_tools/meshes/robot/A_r8.STL" />
+          filename="file://$(find gazebo_tools)/meshes/robot/A_r8.STL" />
+      </geometry>
+      <material
+        name="">
+        <color
+          rgba="0.792156862745098 0.819607843137255 0.933333333333333 1" />
+      </material>
+    </visual>
+    <collision>
+      <origin
+        xyz="0 0 0"
+        rpy="0 0 0" />
+      <geometry>
+        <mesh
+          filename="file://$(find gazebo_tools)/meshes/robot/A_r8.STL" />
       </geometry>
     </collision>
@@ -558,11 +578,11 @@
         izz="9.23881987154415E-06" />
     </inertial>
-    <visual>
-      <origin
-        xyz="0 0 0"
-        rpy="0 0 0" />
-      <geometry>
-        <mesh
-          filename="package://gazebo_tools/meshes/robot/BackRight_wheel.STL" />
+    <!-- <visual>
+      <origin
+        xyz="0 0 0"
+        rpy="0 0 0" />
+      <geometry>
+        <mesh
+          filename="file://$(find gazebo_tools)/meshes/robot/BackRight_wheel.STL" />
       </geometry>
       <material
@@ -571,12 +591,26 @@
           rgba="0.752941176470588 0.752941176470588 0.752941176470588 1" />
       </material>
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