Commit message: last update

File: ws/install/gazebo_tools/share/gazebo_tools/description/BaseMecanumURDF.urdf.xacro (robot description, xacro)
@@ -1 +1,2002 @@
-/ieee_simulation/ws/build/gazebo_tools/description/BaseMecanumURDF.urdf.xacro
+<?xml version="1.0" encoding="utf-8"?>
+<!-- This URDF was automatically created by SolidWorks to URDF Exporter! Originally created by Stephen Brawner (brawner@gmail.com)
+     Commit Version: 1.6.0-4-g7f85cfe  Build Version: 1.6.7995.38578
+     For more information, please see http://wiki.ros.org/sw_urdf_exporter -->
+<robot
+  name="BaseMecanumURDF">
+    <link name="odom">
+      <visual>
+        <origin xyz="0.0 0.0 0.0" rpy="0 0 0" />
+        <geometry>
+          <box size="0.1 0.1 0.1" />
+        </geometry>
+      </visual>
+    <collision>
+      <origin xyz="0.0 0.0 0.0" rpy="0 0 0" />
+      <geometry>
+        <box size="0.1 0.1 0.1" />
+      </geometry>
+    </collision>
+  </link>
+  <!-- Joint to connect odom and base_link -->
+  <joint name="odom_to_base_link" type="fixed">
+    <parent link="odom" />
+    <child link="base_link" />
+    <origin xyz="0.0 0.0 0.0" rpy="0 0 0" />
+  </joint>
+  <link
+    name="base_link">
+    <inertial>
+      <origin
+        xyz="-0.000222645088332468 0.0212706525268758 0.0478471444162569"
+        rpy="0 0 0" />
+      <mass
+        value="1.14473814613392" />
+      <inertia
+        ixx="0.00406802532833408"
+        ixy="-2.59714279495066E-07"
+        ixz="-5.52464867857707E-08"
+        iyy="0.00104621445375526"
+        iyz="8.96167718563971E-05"
+        izz="0.00444895141676235" />
+    </inertial>
+    <visual>
+      <origin
+        xyz="0 0 0"
+        rpy="0 0 0" />
+      <geometry>
+        <mesh
+          filename="package://gazebo_tools/meshes/robot/base_link.STL" />
+      </geometry>
+      <material
+        name="">
+        <color
+          rgba="0.752941176470588 0.752941176470588 0.752941176470588 1" />
+      </material>
+    </visual>
+    <collision>
+      <origin
+        xyz="0 0 0"
+        rpy="0 0 0" />
+      <geometry>
+        <mesh
+          filename="package://gazebo_tools/meshes/robot/base_link.STL" />
+      </geometry>
+    </collision>
+  </link>
+  <link
+    name="FrontRight_wheel">
+    <inertial>
+      <origin
+        xyz="-0.0200915998046353 -4.09353535379131E-05 -7.3187470010113E-05"
+        rpy="0 0 0" />
+      <mass
+        value="0.0641393198112098" />
+      <inertia
+        ixx="1.05909175225007E-05"
+        ixy="-2.65960923461101E-08"
+        ixz="1.4884879064518E-08"
+        iyy="9.22024127424863E-06"
+        iyz="-3.32779596876557E-08"
+        izz="9.1793540218031E-06" />
+    </inertial>
+    <visual>
+      <origin xyz="0 0 0" rpy="0 1.5708 0" />
+      <geometry>
+        <cylinder radius="0.04" length="0.03" />
+      </geometry>
+      <material name="">
+        <color rgba="0.752941176470588 0.752941176470588 0.752941176470588 1" />
+      </material>
+    </visual>
+    <collision>
+      <origin xyz="0 0 0" rpy="0 1.5708 0" />
+      <geometry>
+        <cylinder radius="0.04" length="0.03" />
+      </geometry>
+      <material name="">
+        <color rgba="0.752941176470588 0.752941176470588 0.752941176470588 1" />
+      </material>
+    </collision>
+  </link>
+  <joint
+    name="A_wheel"
+    type="continuous">
+    <origin
+      xyz="-0.092408 -0.0225 0.0375"
+      rpy="1.5773 0 0" />
+    <parent
+      link="base_link" />
+    <child
+      link="FrontRight_wheel" />
+    <axis
+      xyz="1 0 0" />
+  </joint>
+  <link
+    name="A_r1">
+    <inertial>
+      <origin
+        xyz="-0.0200916046432381 0.00815698765209493 -0.0288697688325274"
+        rpy="0 0 0" />
+      <mass
+        value="0.00600569680327048" />
+      <inertia
+        ixx="4.16201839265504E-07"
+        ixy="-2.33787813314613E-07"
+        ixz="-6.6055406175231E-08"
+        iyy="4.34162277016352E-07"
+        iyz="-6.35668102139208E-08"
+        izz="6.41181843474001E-07" />
+    </inertial>
+    <visual>
+      <origin
+        xyz="0 0 0"
+        rpy="0 0 0" />
+      <geometry>
+        <mesh
+          filename="package://gazebo_tools/meshes/robot/A_r1.STL" />
+      </geometry>
+      <material
+        name="">
+        <color
+          rgba="0.792156862745098 0.819607843137255 0.933333333333333 1" />
+      </material>
+    </visual>
+    <collision>
+      <origin
+        xyz="0 0 0"
+        rpy="0 0 0" />
+      <geometry>
+        <mesh
+          filename="package://gazebo_tools/meshes/robot/A_r1.STL" />
+      </geometry>
+    </collision>
+  </link>
+  <joint
+    name="A1"
+    type="continuous">
+    <origin
+      xyz="0 0 0"
+      rpy="0 0 0" />
+    <parent
+      link="FrontRight_wheel" />
+    <child
+      link="A_r1" />
+    <axis
+      xyz="-0.70711 -0.68047 -0.19226" />
+  </joint>
+  <link
+    name="A_r2">
+    <inertial>
+      <origin
+        xyz="-0.0200916046432381 -0.0146461480299166 -0.0261818705956196"
+        rpy="0 0 0" />
+      <mass
+        value="0.00600569680327048" />
+      <inertia
+        ixx="4.16201839265597E-07"
+        ixy="-2.1202117379408E-07"
+        ixz="1.18604722512999E-07"
+        iyy="4.74105250031347E-07"
+        iyz="1.03509783228825E-07"
+        izz="6.01238870459196E-07" />
+    </inertial>
+    <visual>
+      <origin
+        xyz="0 0 0"
+        rpy="0 0 0" />
+      <geometry>
+        <mesh
+          filename="package://gazebo_tools/meshes/robot/A_r2.STL" />
+      </geometry>
+      <material
+        name="">
+        <color
+          rgba="0.792156862745098 0.819607843137255 0.933333333333333 1" />
+      </material>
+    </visual>
+    <collision>
+      <origin
+        xyz="0 0 0"
+        rpy="0 0 0" />
+      <geometry>
+        <mesh
+          filename="package://gazebo_tools/meshes/robot/A_r2.STL" />
+      </geometry>
+    </collision>
+  </link>
+  <joint
+    name="A2"
+    type="continuous">
+    <origin
+      xyz="0 0 0"
+      rpy="0 0 0" />
+    <parent
+      link="FrontRight_wheel" />
+    <child
+      link="A_r2" />
+    <axis
+      xyz="-0.70711 -0.61711 0.34521" />
+  </joint>
+  <link
+    name="A_r3">
+    <inertial>
+      <origin
+        xyz="-0.0200916046432382 -0.0261818705956195 0.0146461480299167"
+        rpy="0 0 0" />
+      <mass
+        value="0.00600569680327051" />
+      <inertia
+        ixx="4.16201839266206E-07"
+        ixy="1.18604722512901E-07"
+        ixz="2.12021173793902E-07"
+        iyy="6.01238870459649E-07"
+        iyz="-1.03509783228739E-07"
+        izz="4.74105250031909E-07" />
+    </inertial>
+    <visual>
+      <origin
+        xyz="0 0 0"
+        rpy="0 0 0" />
+      <geometry>
+        <mesh
+          filename="package://gazebo_tools/meshes/robot/A_r3.STL" />
+      </geometry>
+      <material
+        name="">
+        <color
+          rgba="0.792156862745098 0.819607843137255 0.933333333333333 1" />
+      </material>
+    </visual>
+    <collision>
+      <origin
+        xyz="0 0 0"
+        rpy="0 0 0" />
+      <geometry>
+        <mesh
+          filename="package://gazebo_tools/meshes/robot/A_r3.STL" />
+      </geometry>
+    </collision>
+  </link>
+  <joint
+    name="A3"
+    type="continuous">
+    <origin
+      xyz="0 0 0"
+      rpy="0 0 0" />
+    <parent
+      link="FrontRight_wheel" />
+    <child
+      link="A_r3" />
+    <axis
+      xyz="-0.70711 0.34521 0.61711" />
+  </joint>
+  <link
+    name="A_r4">
+    <inertial>
+      <origin
+        xyz="-0.0200916046432381 0.0146461480299168 0.0261818705956195"
+        rpy="0 0 0" />
+      <mass
+        value="0.00600569680327057" />
+      <inertia
+        ixx="4.16201839266947E-07"
+        ixy="2.12021173793702E-07"
+        ixz="-1.1860472251279E-07"
+        iyy="4.74105250032596E-07"
+        iyz="1.03509783228641E-07"
+        izz="6.01238870460215E-07" />
+    </inertial>
+    <visual>
+      <origin
+        xyz="0 0 0"
+        rpy="0 0 0" />
+      <geometry>
+        <mesh
+          filename="package://gazebo_tools/meshes/robot/A_r4.STL" />
+      </geometry>
+      <material
+        name="">
+        <color
+          rgba="0.792156862745098 0.819607843137255 0.933333333333333 1" />
+      </material>
+    </visual>
+    <collision>
+      <origin
+        xyz="0 0 0"
+        rpy="0 0 0" />
+      <geometry>
+        <mesh
+          filename="package://gazebo_tools/meshes/robot/A_r4.STL" />
+      </geometry>
+    </collision>
+  </link>
+  <joint
+    name="A4"
+    type="continuous">
+    <origin
+      xyz="0 0 0"
+      rpy="0 0 0" />
+    <parent
+      link="FrontRight_wheel" />
+    <child
+      link="A_r4" />
+    <axis
+      xyz="-0.70711 0.61711 -0.34521" />
+  </joint>
+  <link
+    name="A_r5">
+    <inertial>
+      <origin
+        xyz="-0.0200916046432382 0.0261818705956195 -0.0146461480299169"
+        rpy="0 0 0" />
+      <mass
+        value="0.00600569680327054" />
+      <inertia
+        ixx="4.16201839266459E-07"
+        ixy="-1.18604722512857E-07"
+        ixz="-2.1202117379382E-07"
+        iyy="6.01238870459831E-07"
+        iyz="-1.035097832287E-07"
+        izz="4.74105250032141E-07" />
+    </inertial>
+    <visual>
+      <origin
+        xyz="0 0 0"
+        rpy="0 0 0" />
+      <geometry>
+        <mesh
+          filename="package://gazebo_tools/meshes/robot/A_r5.STL" />
+      </geometry>
+      <material
+        name="">
+        <color
+          rgba="0.792156862745098 0.819607843137255 0.933333333333333 1" />
+      </material>
+    </visual>
+    <collision>
+      <origin
+        xyz="0 0 0"
+        rpy="0 0 0" />
+      <geometry>
+        <mesh
+          filename="package://gazebo_tools/meshes/robot/A_r5.STL" />
+      </geometry>
+    </collision>
+  </link>
+  <joint
+    name="A5"
+    type="continuous">
+    <origin
+      xyz="0 0 0"
+      rpy="0 0 0" />
+    <parent
+      link="FrontRight_wheel" />
+    <child
+      link="A_r5" />
+    <axis
+      xyz="-0.70711 -0.34521 -0.61711" />
+  </joint>
+  <link
+    name="A_r6">
+    <inertial>
+      <origin
+        xyz="-0.0200916046432382 -0.0288697688325274 -0.00815698765209482"
+        rpy="0 0 0" />
+      <mass
+        value="0.00600569680327051" />
+      <inertia
+        ixx="4.16201839265985E-07"
+        ixy="-6.60554061751913E-08"
+        ixz="2.33787813314476E-07"
+        iyy="6.41181843474351E-07"
+        iyz="6.35668102138827E-08"
+        izz="4.34162277016823E-07" />
+    </inertial>
+    <visual>
+      <origin
+        xyz="0 0 0"
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
File: ws/install/gazebo_tools/share/gazebo_tools/description/BaseMecanumURDF_old.urdf.xacro (robot description, xacro)
@@ -1 +1,2085 @@
-/ieee_simulation/ws/build/gazebo_tools/description/BaseMecanumURDF_old.urdf.xacro
+<?xml version="1.0" encoding="utf-8"?>
+<!-- This URDF was automatically created by SolidWorks to URDF Exporter! Originally created by Stephen Brawner (brawner@gmail.com)
+     Commit Version: 1.6.0-4-g7f85cfe  Build Version: 1.6.7995.38578
+     For more information, please see http://wiki.ros.org/sw_urdf_exporter -->
+<robot
+  name="BaseMecanumURDF">
+    <link name="odom">
+      <visual>
+        <origin xyz="0.0 0.0 0.0" rpy="0 0 0" />
+      </visual>
+  </link>
+  <!-- Joint to connect odom and base_link -->
+  <joint name="odom_to_base_link" type="fixed">
+    <parent link="odom" />
+    <child link="base_link" />
+    <origin xyz="0.0 0.0 0.0" rpy="0 0 0" />
+  </joint>
+  <link
+    name="base_link">
+    <inertial>
+      <origin
+        xyz="-0.000222645088332468 0.0212706525268758 0.0478471444162569"
+        rpy="0 0 0" />
+      <mass
+        value="1.14473814613392" />
+      <inertia
+        ixx="0.00406802532833408"
+        ixy="-2.59714279495066E-07"
+        ixz="-5.52464867857707E-08"
+        iyy="0.00104621445375526"
+        iyz="8.96167718563971E-05"
+        izz="0.00444895141676235" />
+    </inertial>
+    <visual>
+      <origin
+        xyz="0 0 0"
+        rpy="0 0 0" />
+      <geometry>
+        <mesh
+          filename="file://$(find gazebo_tools)/meshes/robot/base_link.STL" />
+      </geometry>
+      <material
+        name="">
+        <color
+          rgba="0.752941176470588 0.752941176470588 0.752941176470588 1" />
+      </material>
+    </visual>
+    <collision>
+      <origin
+        xyz="0 0 0"
+        rpy="0 0 0" />
+      <geometry>
+        <mesh
+          filename="file://$(find gazebo_tools)/meshes/robot/base_link.STL" />
+      </geometry>
+    </collision>
+  </link>
+  <link
+    name="FrontRight_wheel">
+    <inertial>
+      <origin
+        xyz="-0.0200915998046353 -4.09353535379131E-05 -7.3187470010113E-05"
+        rpy="0 0 0" />
+      <mass
+        value="0.0641393198112098" />
+      <inertia
+        ixx="1.05909175225007E-05"
+        ixy="-2.65960923461101E-08"
+        ixz="1.4884879064518E-08"
+        iyy="9.22024127424863E-06"
+        iyz="-3.32779596876557E-08"
+        izz="9.1793540218031E-06" />
+    </inertial>
+    <!-- <inertial>
+      <origin xyz="0 0 0" rpy="0 0 0" />
+      <mass value="0.0641393198112098" />
+      <inertia
+        ixx="0.0001"
+        ixy="0"
+        ixz="0"
+        iyy="0.0001"
+        iyz="0"
+        izz="0.0001" />
+    </inertial> -->
+    <!-- <visual>
+      <origin
+        xyz="0 0 0"
+        rpy="0 0 0" />
+      <geometry>
+        <mesh
+          filename="file://$(find gazebo_tools)/meshes/robot/FrontRight_wheel.STL" />
+      </geometry>
+      <material
+        name="">
+        <color
+          rgba="0.752941176470588 0.752941176470588 0.752941176470588 1" />
+      </material>
+    </visual>  -->
+    <!-- <collision>
+      <origin
+        xyz="-0.0200915998046353 -4.09353535379131E-05 -7.3187470010113E-05"
+        rpy="0 0 0" />
+       <geometry>
+        <mesh
+          filename="file://$(find gazebo_tools)/meshes/robot/FrontRight_wheel.STL" />
+      </geometry>
+      <geometry>
+        <cylinder radius="0.05" length="0.1"/>
+      </geometry>
+       <box size="0.5 0.3 0.1"/>
+    </collision> -->
+    <visual>
+      <origin
+        xyz="-0.02 0 0"
+        rpy="0 1.5708 0" />
+      <geometry>
+        <cylinder radius="0.04" length="0.03"/>
+      </geometry>
+    </visual>
+    <collision>
+      <origin xyz="0 0 0" rpy="0 0 0" />
+      <geometry>
+        <box size="0.04 0.04 0.04"/>
+      </geometry>
+    </collision>
+  </link>
+  <joint
+    name="A_wheel"
+    type="continuous">
+    <origin
+      xyz="-0.092408 -0.0225 0.0375"
+      rpy="1.5773 0 0" />
+    <parent
+      link="base_link" />
+    <child
+      link="FrontRight_wheel" />
+    <axis
+      xyz="1 0 0" />
+  </joint>
+  <link
+    name="A_r1">
+    <inertial>
+      <origin
+        xyz="-0.0200916046432381 0.00815698765209493 -0.0288697688325274"
+        rpy="0 0 0" />
+      <mass
+        value="0.00600569680327048" />
+      <inertia
+        ixx="4.16201839265504E-07"
+        ixy="-2.33787813314613E-07"
+        ixz="-6.6055406175231E-08"
+        iyy="4.34162277016352E-07"
+        iyz="-6.35668102139208E-08"
+        izz="6.41181843474001E-07" />
+    </inertial>
+    <visual>
+      <origin
+        xyz="0 0 0"
+        rpy="0 0 0" />
+      <geometry>
+        <mesh
+          filename="file://$(find gazebo_tools)/meshes/robot/A_r1.STL" />
+      </geometry>
+      <material
+        name="">
+        <color
+          rgba="0.792156862745098 0.819607843137255 0.933333333333333 1" />
+      </material>
+    </visual>
+    <collision>
+      <origin
+        xyz="0 0 0"
+        rpy="0 0 0" />
+      <geometry>
+        <mesh
+          filename="file://$(find gazebo_tools)/meshes/robot/A_r1.STL" />
+      </geometry>
+    </collision>
+  </link>
+  <joint
+    name="A1"
+    type="continuous">
+    <origin
+      xyz="0 0 0"
+      rpy="0 0 0" />
+    <parent
+      link="FrontRight_wheel" />
+    <child
+      link="A_r1" />
+    <axis
+      xyz="-0.70711 -0.68047 -0.19226" />
+  </joint>
+  <link
+    name="A_r2">
+    <inertial>
+      <origin
+        xyz="-0.0200916046432381 -0.0146461480299166 -0.0261818705956196"
+        rpy="0 0 0" />
+      <mass
+        value="0.00600569680327048" />
+      <inertia
+        ixx="4.16201839265597E-07"
+        ixy="-2.1202117379408E-07"
+        ixz="1.18604722512999E-07"
+        iyy="4.74105250031347E-07"
+        iyz="1.03509783228825E-07"
+        izz="6.01238870459196E-07" />
+    </inertial>
+    <visual>
+      <origin
+        xyz="0 0 0"
+        rpy="0 0 0" />
+      <geometry>
+        <mesh
+          filename="file://$(find gazebo_tools)/meshes/robot/A_r2.STL" />
+      </geometry>
+      <material
+        name="">
+        <color
+          rgba="0.792156862745098 0.819607843137255 0.933333333333333 1" />
+      </material>
+    </visual>
+    <collision>
+      <origin
+        xyz="0 0 0"
+        rpy="0 0 0" />
+      <geometry>
+        <mesh
+          filename="file://$(find gazebo_tools)/meshes/robot/A_r2.STL" />
+      </geometry>
+    </collision>
+  </link>
+  <joint
+    name="A2"
+    type="continuous">
+    <origin
+      xyz="0 0 0"
+      rpy="0 0 0" />
+    <parent
+      link="FrontRight_wheel" />
+    <child
+      link="A_r2" />
+    <axis
+      xyz="-0.70711 -0.61711 0.34521" />
+  </joint>
+  <link
+    name="A_r3">
+    <inertial>
+      <origin
+        xyz="-0.0200916046432382 -0.0261818705956195 0.0146461480299167"
+        rpy="0 0 0" />
+      <mass
+        value="0.00600569680327051" />
+      <inertia
+        ixx="4.16201839266206E-07"
+        ixy="1.18604722512901E-07"
+        ixz="2.12021173793902E-07"
+        iyy="6.01238870459649E-07"
+        iyz="-1.03509783228739E-07"
+        izz="4.74105250031909E-07" />
+    </inertial>
+    <visual>
+      <origin
+        xyz="0 0 0"
+        rpy="0 0 0" />
+      <geometry>
+        <mesh
+          filename="file://$(find gazebo_tools)/meshes/robot/A_r3.STL" />
+      </geometry>
+      <material
+        name="">
+        <color
+          rgba="0.792156862745098 0.819607843137255 0.933333333333333 1" />
+      </material>
+    </visual>
+    <collision>
+      <origin
+        xyz="0 0 0"
+        rpy="0 0 0" />
+      <geometry>
+        <mesh
+          filename="file://$(find gazebo_tools)/meshes/robot/A_r3.STL" />
+      </geometry>
+    </collision>
+  </link>
+  <joint
+    name="A3"
+    type="continuous">
+    <origin
+      xyz="0 0 0"
+      rpy="0 0 0" />
+    <parent
+      link="FrontRight_wheel" />
+    <child
+      link="A_r3" />
+    <axis
+      xyz="-0.70711 0.34521 0.61711" />
+  </joint>
+  <link
+    name="A_r4">
+    <inertial>
+      <origin
+        xyz="-0.0200916046432381 0.0146461480299168 0.0261818705956195"
+        rpy="0 0 0" />
+      <mass
+        value="0.00600569680327057" />
+      <inertia
+        ixx="4.16201839266947E-07"
+        ixy="2.12021173793702E-07"
+        ixz="-1.1860472251279E-07"
+        iyy="4.74105250032596E-07"
+        iyz="1.03509783228641E-07"
+        izz="6.01238870460215E-07" />
+    </inertial>
+    <visual>
+      <origin
+        xyz="0 0 0"
+        rpy="0 0 0" />
+      <geometry>
+        <mesh
+          filename="file://$(find gazebo_tools)/meshes/robot/A_r4.STL" />
+      </geometry>
+      <material
+        name="">
+        <color
+          rgba="0.792156862745098 0.819607843137255 0.933333333333333 1" />
+      </material>
+    </visual>
+    <collision>
+      <origin
+        xyz="0 0 0"
+        rpy="0 0 0" />
+      <geometry>
+        <mesh
+          filename="file://$(find gazebo_tools)/meshes/robot/A_r4.STL" />
+      </geometry>
+    </collision>
+  </link>
+  <joint
+    name="A4"
+    type="continuous">
+    <origin
+      xyz="0 0 0"
+      rpy="0 0 0" />
+    <parent
+      link="FrontRight_wheel" />
+    <child
+      link="A_r4" />
+    <axis
+      xyz="-0.70711 0.61711 -0.34521" />
+  </joint>
+  <link
+    name="A_r5">
+    <inertial>
+      <origin
+        xyz="-0.0200916046432382 0.0261818705956195 -0.0146461480299169"
+        rpy="0 0 0" />
+      <mass
+        value="0.00600569680327054" />
+      <inertia
+        ixx="4.16201839266459E-07"
+        ixy="-1.18604722512857E-07"
+        ixz="-2.1202117379382E-07"
+        iyy="6.01238870459831E-07"
+        iyz="-1.035097832287E-07"
+        izz="4.74105250032141E-07" />
+    </inertial>
+    <visual>
+      <origin
+        xyz="0 0 0"
+        rpy="0 0 0" />
+      <geometry>
+        <mesh
+          filename="file://$(find gazebo_tools)/meshes/robot/A_r5.STL" />
+      </geometry>
+      <material
+        name="">
+        <color
+          rgba="0.792156862745098 0.819607843137255 0.933333333333333 1" />
+      </material>
+    </visual>
+    <collision>
+      <origin
+        xyz="0 0 0"
+        rpy="0 0 0" />
+      <geometry>
+        <mesh
+          filename="file://$(find gazebo_tools)/meshes/robot/A_r5.STL" />
+      </geometry>
+    </collision>
+  </link>
+  <joint
+    name="A5"
+    type="continuous">
+    <origin
+      xyz="0 0 0"
+      rpy="0 0 0" />
+    <parent
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